Commit message: add robot control

File: urdf/sisbot.urdf (robot description, URDF)
Before this commit: robot sisbot, 19 links, 18 joints
Joints:
- joint robotiq_85_left_knuckle_joint: limit lower=0 upper=0.8575 effort=1000 velocity=2.0 -> lower=0 upper=0.343 effort=1000 velocity=2.0
- joint shoulder_lift_joint: limit lower=-6.28318530718 upper=6.28318530718 effort=150.0 velocity=3.15 -> lower=-3.14159265359 upper=3.14159265359 effort=150.0 velocity=3.15
- joint shoulder_pan_joint: limit lower=-6.28318530718 upper=6.28318530718 effort=150.0 velocity=3.15 -> lower=-3.14159265359 upper=3.14159265359 effort=150.0 velocity=3.15
- joint world_joint: origin xyz=0.0 0.0 0.0 rpy=0.0 0.0 0.0 -> xyz=0.0 0.0 0.1 rpy=0.0 0.0 -0.6
- joint wrist_1_joint: limit lower=-6.28318530718 upper=6.28318530718 effort=28.0 velocity=3.2 -> lower=-3.14159265359 upper=3.14159265359 effort=28.0 velocity=3.2
- joint wrist_2_joint: limit lower=-6.28318530718 upper=6.28318530718 effort=28.0 velocity=3.2 -> lower=-3.14159265359 upper=3.14159265359 effort=28.0 velocity=3.2
- joint wrist_3_joint: limit lower=-6.28318530718 upper=6.28318530718 effort=28.0 velocity=3.2 -> lower=-3.14159265359 upper=3.14159265359 effort=28.0 velocity=3.2

Commit message: sisbot basic control done

File: urdf/sisbot.urdf (robot description, URDF)
Before this commit: robot sisbot, 19 links, 18 joints
Links:
- link forearm_link: geometry collision mesh filename=../meshes/ur5/collision/forearm.stl; visual mesh filename=../meshes/ur5/visual/forearm.obj
- link shoulder_link: geometry collision mesh filename=../meshes/ur5/collision/shoulder.stl; visual mesh filename=../meshes/ur5/visual/shoulder.obj
- link upper_arm_link: geometry collision mesh filename=../meshes/ur5/collision/upperarm.stl; visual mesh filename=../meshes/ur5/visual/upperarm.obj
- link wrist_1_link: geometry collision mesh filename=../meshes/ur5/collision/wrist1.stl; visual mesh filename=../meshes/ur5/visual/wrist1.obj
- link wrist_2_link: geometry collision mesh filename=../meshes/ur5/collision/wrist2.stl; visual mesh filename=../meshes/ur5/visual/wrist2.obj
- link wrist_3_link: geometry collision mesh filename=../meshes/ur5/collision/wrist3.stl; visual mesh filename=../meshes/ur5/visual/wrist3.obj
Joints:
- joint world_joint: origin xyz=0.0 0.0 0.1 rpy=0.0 0.0 -0.6 -> xyz=0.0 0.0 0.7 rpy=0.0 0.0 -0.6

Commit message: 12/7 go home

File: urdf/sisbot.urdf (robot description, URDF)
Before this commit: robot sisbot, 19 links, 18 joints
Links:
- link base_link: geometry collision mesh filename=../meshes/ur5/collision/base.stl; visual mesh filename=../meshes/ur5/visual/base.obj
Joints:
- joint world_joint: origin xyz=0.0 0.0 0.7 rpy=0.0 0.0 -0.6 -> xyz=0.0 0.0 0.1 rpy=0.0 0.0 -0.6

Commit message: working on grasping

File: urdf/sisbot.urdf (robot description, URDF)
Before this commit: robot sisbot, 19 links, 18 joints
Joints:
- joint world_joint: origin xyz=0.0 0.0 0.1 rpy=0.0 0.0 -0.6 -> xyz=0.0 0.0 0.1 rpy=0.0 0.0 0
